File: Esp_4relay_feedback.brd (EAGLE design)
At the start: 150 x 100 mm, 106 parts, among them IC1 LM1117MP-3.3, IC2 NE555, K1 G5LE, K2 G5LE, K3 G5LE, K4 G5LE, K5 G5LE, K6 G5LE, K7 G5LE, K8 G5LE, Q1 16MHz, Q10 BC547, Q11 TIP120, Q2 BC547, Q4 BC547, Q5 BC547, Q6 BC547, Q7 BC547, Q8 BC547, Q9 BC547, T1 2N7000, T2 2N7000, U2 ATMEGA328P_PDIP

Commit message: Signed-off-by: amitkawade47 <amitkawade47@gmail.com>
Parts:
- moved U$2 1.00 mm to (184.0, 21.0)
Changed lines of the file:
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@@
 <element name="R36" library="amit_rcl" package="0207/5V" value="10k" x="227" y="40" rot="R270"/>
 <element name="R37" library="amit_rcl" package="0207/5V" value="10k" x="228" y="60" rot="R90"/>
-<element name="U$2" library="amit_high_link_5W" package="AMIT_HIGH_LINK" value="AMIT_HIGH_LINK" x="185" y="21" rot="R90"/>
+<element name="U$2" library="amit_high_link_5W" package="AMIT_HIGH_LINK" value="AMIT_HIGH_LINK" x="184" y="21" rot="R90"/>
 <element name="X9" library="amit_screw_terminal_23" package="W237-102" value="" x="167" y="6">
 <attribute name="OC_NEWARK" value="70K9898" x="167" y="6" size="1.778" layer="27" display="off"/>
@@
 <wire x1="162.19" y1="41.73" x2="152" y2="38" width="0" layer="19" extent="1-1"/>
 <wire x1="169.81" y1="44.27" x2="162.19" y2="41.73" width="0" layer="19" extent="1-1"/>
-<wire x1="175.93" y1="36.48" x2="169.81" y2="44.27" width="0" layer="19" extent="1-1"/>
+<wire x1="174.93" y1="36.48" x2="169.81" y2="44.27" width="0" layer="19" extent="1-1"/>
 <wire x1="161" y1="18.27" x2="152" y2="35" width="0" layer="19" extent="1-1"/>
 <wire x1="155.81" y1="15.81" x2="161" y2="18.27" width="0" layer="19" extent="1-1"/>
 <wire x1="154.27" y1="4" x2="155.81" y2="15.81" width="0" layer="19" extent="1-1"/>
 <wire x1="148" y1="1.73" x2="154.27" y2="4" width="0" layer="19" extent="1-1"/>
-<wire x1="202.27" y1="44.81" x2="175.93" y2="36.48" width="0" layer="19" extent="1-1"/>
+<wire x1="202.27" y1="44.81" x2="174.93" y2="36.48" width="0" layer="19" extent="1-1"/>
 <wire x1="210.46" y1="41.4484" x2="202.27" y2="44.81" width="0" layer="19" extent="1-1"/>
 <wire x1="210.73" y1="55.19" x2="211.963" y2="42.9514" width="0" layer="19" extent="1-1"/>
@@
 <wire x1="168.35" y1="19.54" x2="169.81" y2="39.19" width="0" layer="19" extent="1-1"/>
 <wire x1="155.829" y1="9.9568" x2="168.35" y2="19.54" width="0" layer="19" extent="16-16"/>
-<wire x1="193.93" y1="36.48" x2="169.81" y2="39.19" width="0" layer="19" extent="1-1"/>
+<wire x1="192.93" y1="36.48" x2="169.81" y2="39.19" width="0" layer="19" extent="1-1"/>
 <wire x1="116.0526" y1="54.991" x2="158" y2="61.08" width="0" layer="19" extent="1-1"/>
 </signal>
@@
 <contactref element="U$2" pad="AC1"/>
 <contactref element="X9" pad="1"/>
-<wire x1="164.5" y1="4.73" x2="181.93" y2="2.88" width="0" layer="19" extent="1-1"/>
+<wire x1="164.5" y1="4.73" x2="180.93" y2="2.88" width="0" layer="19" extent="1-1"/>
 <wire x1="111.5314" y1="59.7154" x2="164.5" y2="4.73" width="0" layer="19" extent="1-1"/>
 </signal>
@@
 </signal>
 <signal name="N$83">
-<via x="181.2544" y="10.0076" extent="1-16" drill="1" diameter="1.016" shape="square"/>
+<via x="167.2544" y="15.0076" extent="1-16" drill="1" diameter="1.016" shape="square"/>
 </signal>
 <signal name="N$84">
@@
 </signal>
 <signal name="N$104">
-<via x="183.5404" y="15.6718" extent="1-16" drill="1" diameter="1.4224" shape="square"/>
+<via x="169.5404" y="19.6718" extent="1-16" drill="1" diameter="1.4224" shape="square"/>
 </signal>
 <signal name="N$66">
 <contactref element="U$2" pad="AC2"/>
 <contactref element="X9" pad="2"/>
-<wire x1="169.5" y1="4.73" x2="187.93" y2="2.88" width="0" layer="19" extent="1-1"/>
+<wire x1="169.5" y1="4.73" x2="186.93" y2="2.88" width="0" layer="19" extent="1-1"/>
 </signal>
 </signals>
